File: Electrical/pcb/pcb.kicad_sch (KiCad schematic)
At the start: 8 parts, among them U1 LM2917N-8/NOPB

Commit message: changes
Parts:
- added C3: 20nF, Capacitor_THT:CP_Radial_D5.0mm_P2.00mm, symbol Device:C_Polarized_Small_US
- added C4: 1uF, Capacitor_THT:CP_Radial_D5.0mm_P2.00mm, symbol Device:C_Polarized_Small_US
- added R2: 100k, Resistor_THT:R_Axial_DIN0207_L6.3mm_D2.5mm_P10.16mm_Horizontal, symbol PCM_SL_Resistors:100k
- added Rload2: 10k, Resistor_THT:R_Axial_DIN0207_L6.3mm_D2.5mm_P10.16mm_Horizontal, symbol PCM_SL_Resistors:100k
- added Rpower2: 470, Resistor_THT:R_Axial_DIN0207_L6.3mm_D2.5mm_P10.16mm_Horizontal, symbol PCM_SL_Resistors:100k
- added U2: LM2917N-8/NOPB, N08E_TEX, symbol 2024-11-06_18-44-41:LM2917N-8_NOPB
Connections:
- net +12V: now also Rpower2.2, U2.5 (COL)
- net GND: now also C3.2, C4.2, R2.1, Rload2.1, U2.8 (TACH-)
- net at A1.A2: now also Rload2.2, U2.4 (EMIT), U2.7 (IN-)
- net HALL EFFECT SENSOR renamed ENGINE HALL EFFECT SENSOR
- new net: Rpower2.1, U2.6 (V+)
- new net: C3.1, U2.2 (CP)
- new net: C4.1, R2.2, U2.3 (CP/IN+)
- new net OUTPUT HALL EFFECT SENSOR: U2.1 (TACH+)
Other:
- moved on the sheet: A1, A2, C1, C2, R1, Rload1, Rpower1, U1
